File: Hardware/SparkFun_Artemis_OpenLog.sch (EAGLE design)
At the start: 90 parts, among them J14 CORTEX_JTAG, J6 MICRO-SD, Q1 20V/0.2A/8MHz/1.2Ω/1Vth, Q10 20V/0.2A/8MHz/1.2Ω/1Vth, Q2 20V/4.2A/52mΩ/1.4W, Q3 20V/0.2A/8MHz/1.2Ω/1Vth, Q7 20V/0.2A/8MHz/1.2Ω/1Vth, Q9 20V/0.2A/8MHz/1.2Ω/1Vth, U1 3.0V Supervisor, U10 CH340E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

Commit message: Add pull down to Qwiic vreg
Parts:
- added R3: 220k, SparkFun-Resistors:220KOHM-0402T-1/16W-1%
Connections:
- net GND: now also R3.1
- net QWIIC_PWR: now also R3.2
Other:
- note added: "Change from X04 to V10: ICM PWR moved from 22 to 27 SD CS moved from 10 to 23 Add PWR_LED on 29 Add VREG_EN on 25 Add SDIO connection to SD"
- note removed: "Analog to Qwiic VCC"
- note removed: "On v10: ICM PWR moved from 22 to 27 SD CS moved from 10 to 23 Add PWR_LED on 29 Add VREG_EN on 25 Add SDIO connection to SD"
- moved on the sheet: C5, C7, J11, U4

Commit message: Updates as per Paul's work diary. Added RST pad and VIN monitor.
Parts:
- added J7: (no value), SparkFun-Connectors:CONN_01PTH_NO_SILK_YES_STOP
- added R6: 1M, New_Parts:1MOHM-0402T-1/16W-1%
- added R7: 2M, New_Parts:2MOHM-0402T-1/16W-1%
- C5: value 10uF -> 0.1uF; device SparkFun-Capacitors:10UF-0402T-6.3V-20% -> SparkFun-Capacitors:0.1UF-0402T-6.3V-10%-X7R
- R2: value 220k -> 330K; device SparkFun-Resistors:220KOHM-0402T-1/16W-1% -> New_Parts:330KOHM-0402T-1/16W-1%
- renumbered VREG to VE
Connections:
- new net VIN/3: R6.2, R7.1, U8.AD34(CMPRF2/PDMDATA)
- net ARTEMIS_!RESET: now also J7.1
- net GND: now also R6.1
- net VIN: now also R7.2
Other:
- note added: "VIN monitor"
Changed lines of the file:
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@@
 <part name="SUPPLY4" library="SparkFun-PowerSymbols" deviceset="3.3V" device=""/>
 <part name="J3" library="SparkFun-Connectors" deviceset="CONN_02" device="1X02_NO_SILK"/>
-<part name="R2" library="SparkFun-Resistors" deviceset="220KOHM" device="-0402T-1/16W-1%" value="220k"/>
+<part name="R2" library="New_Parts" deviceset="330KOHM" device="-0402T-1/16W-1%" value="330K"/>
 <part name="FRAME1" library="SparkFun-Aesthetics" deviceset="FRAME-LEDGER" device=""/>
 <part name="SUPPLY11" library="SparkFun-PowerSymbols" deviceset="VCC_1" device=""/>
 <part name="D6" library="SparkFun-DiscreteSemi" deviceset="DIODE-SCHOTTKY" device="-BAT20J" value="1A/23V/620mV"/>
-<part name="C5" library="SparkFun-Capacitors" deviceset="10UF" device="-0402T-6.3V-20%" value="10uF"/>
+<part name="C5" library="SparkFun-Capacitors" deviceset="0.1UF" device="-0402T-6.3V-10%-X7R" value="0.1uF"/>
 <part name="GND6" library="SparkFun-PowerSymbols" deviceset="GND" device=""/>
 <part name="Q2" library="SparkFun-DiscreteSemi" deviceset="MOSFET_PCH" device="-DMG2305UX-7" value="20V/4.2A/52mΩ/1.4W"/>
@@
 <part name="GND10" library="SparkFun-PowerSymbols" deviceset="GND" device=""/>
 <part name="GND12" library="SparkFun-PowerSymbols" deviceset="GND" device=""/>
-<part name="VREG" library="SparkFun-Jumpers" deviceset="JUMPER-SMT_2_NO" device="_SILK" package3d_urn="urn:adsk.eagle:package:39279/1" value=""/>
+<part name="VE" library="SparkFun-Jumpers" deviceset="JUMPER-SMT_2_NO" device="_SILK" package3d_urn="urn:adsk.eagle:package:39279/1" value=""/>
 <part name="LOGO3" library="SparkFun-Aesthetics" deviceset="SPECIAL_INSTRUCTIONS" device="-ORDERING"/>
 <part name="LOGO4" library="SparkFun-Aesthetics" deviceset="SFE_LOGO_FLAME" device=".1_INCH"/>
@@
 <part name="R3" library="SparkFun-Resistors" deviceset="220KOHM" device="-0402T-1/16W-1%" value="220k"/>
 <part name="GND9" library="SparkFun-PowerSymbols" deviceset="GND" device=""/>
+<part name="GND13" library="SparkFun-PowerSymbols" deviceset="GND" device=""/>
+<part name="R6" library="New_Parts" deviceset="1MOHM" device="-0402T-1/16W-1%" value="1M"/>
+<part name="R7" library="New_Parts" deviceset="2MOHM" device="-0402T-1/16W-1%" value="2M"/>
+<part name="J7" library="SparkFun-Connectors" deviceset="CONN_01" device="PTH_NO_SILK_YES_STOP"/>
 </parts>
 <sheets>
@@
 <wire x1="388.62" y1="210.82" x2="388.62" y2="279.4" width="0.2032" layer="97" style="longdash"/>
 <wire x1="388.62" y1="68.58" x2="388.62" y2="144.78" width="0.2032" layer="97" style="longdash"/>
+<text x="262.636" y="263.652" size="1.778" layer="97" font="vector">VIN monitor</text>
 </plain>
 <instances>
@@
 <attribute name="VALUE" x="342.9" y="106.426" size="1.778" layer="96" align="top-center"/>
 </instance>
-<instance part="VREG" gate="G$1" x="147.32" y="43.18" smashed="yes">
-<attribute name="NAME" x="144.272" y="39.624" size="1.778" layer="95" font="vector"/>
+<instance part="VE" gate="G$1" x="147.32" y="43.18" smashed="yes">
+<attribute name="NAME" x="146.05" y="39.116" size="1.778" layer="95" font="vector"/>
 <attribute name="VALUE" x="144.78" y="40.64" size="1.778" layer="96" font="vector" align="top-left"/>
 </instance>
@@
 <instance part="GND9" gate="1" x="335.28" y="99.06" smashed="yes">
 <attribute name="VALUE" x="335.28" y="98.806" size="1.778" layer="96" align="top-center"/>
+</instance>
+<instance part="GND13" gate="1" x="271.78" y="226.06" smashed="yes">
+<attribute name="VALUE" x="271.78" y="225.806" size="1.778" layer="96" align="top-center"/>
+</instance>
+<instance part="R6" gate="G$1" x="271.78" y="236.22" smashed="yes" rot="R90">
+<attribute name="NAME" x="270.256" y="236.22" size="1.778" layer="95" font="vector" rot="R90" align="bottom-center"/>
+<attribute name="VALUE" x="273.304" y="236.22" size="1.778" layer="96" font="vector" rot="R90" align="top-center"/>
+</instance>
+<instance part="R7" gate="G$1" x="271.78" y="251.46" smashed="yes" rot="R90">
+<attribute name="NAME" x="270.256" y="251.46" size="1.778" layer="95" font="vector" rot="R90" align="bottom-center"/>
+<attribute name="VALUE" x="273.304" y="251.46" size="1.778" layer="96" font="vector" rot="R90" align="top-center"/>
+</instance>
+<instance part="J7" gate="G$1" x="127" y="187.96" smashed="yes">
+<attribute name="VALUE" x="124.46" y="183.134" size="1.778" layer="96" font="vector"/>
+<attribute name="NAME" x="124.46" y="191.008" size="1.778" layer="95" font="vector"/>
 </instance>
 </instances>
@@
 <wire x1="335.28" y1="101.6" x2="335.28" y2="104.14" width="0.1524" layer="91"/>
 </segment>
+<segment>
+<pinref part="R6" gate="G$1" pin="1"/>
+<pinref part="GND13" gate="1" pin="GND"/>
+<wire x1="271.78" y1="231.14" x2="271.78" y2="228.6" width="0.1524" layer="91"/>
+</segment>
 </net>
 <net name="3.3V" class="0">
@@
 <wire x1="342.9" y1="121.92" x2="342.9" y2="124.46" width="0.1524" layer="91"/>
 <label x="342.9" y="124.46" size="1.27" layer="95" rot="R90" xref="yes"/>
+</segment>
+<segment>
+<pinref part="R7" gate="G$1" pin="2"/>
+<wire x1="271.78" y1="256.54" x2="271.78" y2="259.08" width="0.1524" layer="91"/>
+<wire x1="271.78" y1="259.08" x2="264.16" y2="259.08" width="0.1524" layer="91"/>
+<label x="264.16" y="259.08" size="1.27" layer="95" rot="R180" xref="yes"/>
 </segment>
 </net>
@@
 <pinref part="S3" gate="G$1" pin="2"/>
 </segment>
+<segment>
+<pinref part="J7" gate="G$1" pin="1"/>
+<wire x1="134.62" y1="187.96" x2="139.7" y2="187.96" width="0.1524" layer="91"/>
+<label x="139.7" y="187.96" size="1.27" layer="95" xref="yes"/>
+</segment>
 </net>
 <net name="ARTEMIS_RX0" class="0">
@@
 </segment>
 <segment>
-<pinref part="VREG" gate="G$1" pin="2"/>
+<pinref part="VE" gate="G$1" pin="2"/>
 <wire x1="152.4" y1="43.18" x2="154.94" y2="43.18" width="0.1524" layer="91"/>
 <label x="154.94" y="43.18" size="1.27" layer="95" xref="yes"/>
@@
 <segment>
 <pinref part="U8" gate="U1" pin="(SDA2/MISO2/RX1)~D25"/>
-<pinref part="VREG" gate="G$1" pin="1"/>
+<pinref part="VE" gate="G$1" pin="1"/>
 <wire x1="129.54" y1="43.18" x2="142.24" y2="43.18" width="0.1524" layer="91"/>
+</segment>
+</net>
+<net name="VIN/3" class="0">
+<segment>
+<pinref part="U8" gate="U1" pin="AD34(CMPRF2/PDMDATA)"/>
+<wire x1="60.96" y1="25.4" x2="58.42" y2="25.4" width="0.1524" layer="91"/>
+<label x="58.42" y="25.4" size="1.27" layer="95" rot="R180" xref="yes"/>
+</segment>
+<segment>
+<pinref part="R7" gate="G$1" pin="1"/>
+<wire x1="271.78" y1="246.38" x2="271.78" y2="243.84" width="0.1524" layer="91"/>
+<wire x1="271.78" y1="243.84" x2="266.7" y2="243.84" width="0.1524" layer="91"/>
+<pinref part="R6" gate="G$1" pin="2"/>
+<wire x1="271.78" y1="241.3" x2="271.78" y2="243.84" width="0.1524" layer="91"/>
+<junction x="271.78" y="243.84"/>
+<label x="266.7" y="243.84" size="1.27" layer="95" rot="R180" xref="yes"/>
 </segment>
 </net>
@@
 </sheet>
 </sheets>
+<errors>
+</errors>
 </schematic>
 </drawing>

Commit message: Final tweaks. Ready for panelization.
Other:
- note added: "Change from X04 to V10: ICM PWR moved from 22 to 27 SD CS moved from 10 to 23 Add PWR_LED on 29 Add VREG_EN on 25 Add SDIO connection to SD Add VIN monitor on AD34 (R6/R7) QWIIC_PWR (18) will be active high"
- note added: "LEDs"
- note removed: "Change from X04 to V10: ICM PWR moved from 22 to 27 SD CS moved from 10 to 23 Add PWR_LED on 29 Add VREG_EN on 25 Add SDIO connection to SD"
Changed lines of the file:
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@@
 Add PWR_LED on 29
 Add VREG_EN on 25
-Add SDIO connection to SD</text>
+Add SDIO connection to SD
+Add VIN monitor on AD34 (R6/R7)
+QWIIC_PWR (18) will be active high</text>
 <wire x1="320.04" y1="68.58" x2="388.62" y2="68.58" width="0.2032" layer="97" style="longdash"/>
 <wire x1="388.62" y1="210.82" x2="388.62" y2="279.4" width="0.2032" layer="97" style="longdash"/>
 <wire x1="388.62" y1="68.58" x2="388.62" y2="144.78" width="0.2032" layer="97" style="longdash"/>
 <text x="262.636" y="263.652" size="1.778" layer="97" font="vector">VIN monitor</text>
+<text x="342.9" y="269.24" size="2.54" layer="94" align="center">LEDs</text>
 </plain>
 <instances>

Commit message: Minor SCH tweaks. Replaced the USB-C connector.
Parts:
- J5: device USBC:USB_C5 -> SparkFun-Connectors:USB_C_4-LAYER_PADS
Connections:
- net MICROSD_!CS!/SDIO3 renamed MICROSD_!CS!
- net MISO/SDIO0 renamed MISO
- net MOSI/SDIO-CMD renamed MOSI
- net SCK/SDIO-CLK renamed SCK
- net SDIO1 renamed DAT1
- net SDIO2 renamed DAT2
- net GND: now also J5.SHLD
Other:
- note added: "Close the VE split pad to allow the Artemis to disable the 3.3V regulator (forcing it to run from the RTC battery). This will reduce the sleep current draw by approx. 55μA."
- moved on the sheet: C42, C44, C52, C53, C54, J14, Q1, Q3, Q7, R28, R40, R41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

Commit message: V10 PCB tweaks following design review
Parts:
- added R8: 0, SparkFun-Resistors:0OHM-0402T-1/10W
- added SCL, SDA, TP1: TEST-POINT3, SparkFun-Connectors:TEST-POINT3
Connections:
- new net RTC_BAT+: BT1.+, D3.A, R1.1, TP1.1
- net GND: now also R8.1; no longer J5.SHLD
- net N$1: now also J5.SHLD, R8.2; no longer BT1.+, D3.A, R1.1
- net SCL: now also SCL.1
- net SDA: now also SDA.1
Other:
- note added: "SP6214-1.8V ---------------- Iout (max): 100mA Vin (max): 7.0V Vdrop (max): 250mV Iq: 65uA"
- moved on the sheet: J11

Commit message: Final V10 PCB tweaks!?
Parts:
- added GND, QWIIC_3.3V: TEST-POINTTP_15TH_THRU, SparkFun-Connectors:TEST-POINTTP_15TH_THRU
- SCL, SDA: value TEST-POINT3 -> TEST-POINTTP_15TH_THRU; device SparkFun-Connectors:TEST-POINT3 -> SparkFun-Connectors:TEST-POINTTP_15TH_THRU
- U13: value ICM-20948 -> 9DoF IMU
- U3, U4: value AP2112K -> 3.3V
Connections:
- net ICM-20948-LV_MISO renamed ICM-20948-LV_SDO
- net ICM-20948-LV_MOSI renamed ICM-20948-LV_SDI
- removed net MISO: J6.DAT0/MISO, Q10.D, R49.1, U8.(PDMCLK/SWO)~D22, U8.(SDA0/MISO0/I2SDAT)~D6
- removed net MOSI: J6.CMD/MOSI, Q3.D, U8.(MOSI0/CLKOUT)~D7
- new net SDI: J6.DAT0/SDO, Q10.D, R49.1, U8.(PDMCLK/SWO)~D22, U8.(SDA0/SDI0/I2SDAT)~D6
- new net SDO: J6.CMD/SDI, Q3.D, U8.(SDO0/CLKOUT)~D7
- net ARTEMIS_BOOT: now also U8.~BOOT(SDO5/RX1/32KHZ); no longer U8.~BOOT(MOSI5/RX1/32KHZ)
- net ARTEMIS_RX0: now also U8.~D49(RX0/SDA5/SDI5); no longer U8.~D49(RX0/SDA5/MISO5)
- net GND: now also GND.1
- net ICM_!CS!: now also U8.(SDO4)~D44; no longer U8.(MOSI4)~D44
- net MICROSD_!CS!: now also J6.DAT3/!CS!; no longer J6.DAT3/CS
- net QWIIC_3.3V: now also QWIIC_3.3V.1
- net SDA: now also U8.(SDA1/SDI1/RX1/SCCIO)D9; no longer U8.(SDA1/MISO1/RX1/SCCIO)D9
- net VREG_EN1: now also U8.(SDA2/SDI2/RX1)~D25; no longer U8.(SDA2/MISO2/RX1)~D25
Other:
- note added: "Controller In Peripheral Out (CIPO)"
- note added: "Controller Out Peripheral In (COPI)"
- moved on the sheet: J11, J4, J7, SCL, SDA
