File: Hardware/SparkFun_Artemis_OpenLog/SparkFun_Artemis_OpenLog.kicad_sch (KiCad schematic)
At the start: 92 parts, among them J11 Qwiic_RA, J14 CORTEX_JTAG, J2 Conn_01x02, J3 Conn_01x02, J4 CONN_06NO_SILK_NO_POP, J5 JST_2mm_LiPo, J6 MICRO-SD, J7 CONN_01PTH_NO_SILK_YES_STOP, J8 USB_C_Receptacle, Q2 DMG2305UX, U1 3.0V Supervisor, U10 CH340E, U2 MCP73831, U3 AP2112K-3.3, U4 3.3V, U5 BNO086, U8 ARTEMIS_MODULE, Y1 32.768kHz, Y3 32.768kHz

Commit message: Another save point, update gitignore
Parts:
- C10, C11, C9: footprint SparkFun_Artemis_OpenLog:0402 -> SparkFun-Capacitor:C_0402_1005Metric; symbol SparkFun_Artemis_OpenLog-eagle-import:0.1UF-0402-6.3V-10%-X7R -> SparkFun-Capacitor:0.1uF_0402_16V_10%; PROD_ID CAP-14993 -> CAP-25565; Tolerance (none) -> 10%; Voltage (none) -> 16V
- C2, C7: footprint SparkFun_Artemis_OpenLog:0402-TIGHT -> SparkFun-Capacitor:C_0402_1005Metric; symbol SparkFun_Artemis_OpenLog-eagle-import:2.2UF-0402_TIGHT-10V-10%-X5R -> SparkFun-Capacitor:2.2uF_0402_10V_10%; Tolerance (none) -> 10%; Voltage (none) -> 10V
- C29, C30: footprint SparkFun_Artemis_OpenLog:0402-TIGHT -> SparkFun-Capacitor:C_0402_1005Metric; symbol SparkFun_Artemis_OpenLog-eagle-import:15PF-0402T-50V-5% -> SparkFun-Capacitor:15pF_0402_50V_5%; Tolerance (none) -> 5%; Voltage (none) -> 50V
- C5: footprint SparkFun_Artemis_OpenLog:0402-TIGHT -> SparkFun-Capacitor:C_0402_1005Metric; symbol SparkFun_Artemis_OpenLog-eagle-import:0.1UF-0402T-6.3V-10%-X7R -> SparkFun-Capacitor:0.1uF_0402_16V_10%; PROD_ID CAP-14993 -> CAP-25565; Tolerance (none) -> 10%; Voltage (none) -> 16V
- C6, C8: footprint SparkFun_Artemis_OpenLog:0402-TIGHT -> SparkFun-Capacitor:C_0402_1005Metric; symbol SparkFun_Artemis_OpenLog-eagle-import:22PF-0402T-16V-10% -> SparkFun-Capacitor:22pF_0402_50V_5%; PROD_ID CAP-14674 -> CAP-25012; Tolerance (none) -> 5%; Voltage (none) -> 50V
- D1, D3: value 3A/10V/280mV -> BAT60A; footprint SparkFun_Artemis_OpenLog:SOD-323 -> SparkFun-Semiconductor-Standard:SOD-323; symbol SparkFun_Artemis_OpenLog-eagle-import:DIODE-SCHOTTKY-BAT60A -> SparkFun-DiscreteSemi:D_Schottky_3A_10V_0.28V; IMax (none) -> 3A; VDrop (none) -> 0.28V; VMax (none) -> 10V
- D6: value 1A/23V/620mV -> BAT20J; footprint SparkFun_Artemis_OpenLog:SOD-323 -> SparkFun-Semiconductor-Standard:SOD-323; symbol SparkFun_Artemis_OpenLog-eagle-import:DIODE-SCHOTTKY-BAT20J -> SparkFun-DiscreteSemi:D_Schottky_1A_23V_0.62V; IMax (none) -> 1A; VForward (none) -> 0.62V; VReverse (none) -> 23V
- J14: value CORTEX_JTAG -> SWD; footprint SparkFun_Artemis_OpenLog:2X5-PTH-1.27MM -> SparkFun-Connector:2x05_P1.27mm; symbol SparkFun_Artemis_OpenLog-eagle-import:CORTEX_JTAG_DEBUG_MINIMUM_PTH -> SparkFun-Connector:Debug-Cortex-2x5_P1.27mm; SF_ID (none) -> PRT-15362
- J4: value CONN_06NO_SILK_NO_POP -> Conn_01x06; footprint SparkFun_Artemis_OpenLog:1X06_NO_SILK -> SparkFun-Connector:1x06_P2.54mm; symbol SparkFun_Artemis_OpenLog-eagle-import:CONN_06NO_SILK_NO_POP -> SparkFun-Connector:Conn_01x06_P2.54mm
- J7: value CONN_01PTH_NO_SILK_YES_STOP -> Conn_01x01; footprint SparkFun_Artemis_OpenLog:1X01_NO_SILK -> SparkFun-Connector:1x01_P2.54mm; symbol SparkFun_Artemis_OpenLog-eagle-import:CONN_01PTH_NO_SILK_YES_STOP -> SparkFun-Connector:Conn_01x01_P2.54mm
- R29: value 220KOHM-0402T-1/16W-1% -> 100k; footprint SparkFun_Artemis_OpenLog:0402-TIGHT -> SparkFun-Resistor:R_0402_1005Metric; symbol SparkFun_Artemis_OpenLog-eagle-import:220KOHM-0402T-1/16W-1% -> SparkFun-Resistor:100k_0402; PROD_ID RES-15094 -> RES-25013
- R3: value 220k -> 100k; footprint SparkFun_Artemis_OpenLog:0402-TIGHT -> SparkFun-Resistor:R_0402_1005Metric; symbol SparkFun_Artemis_OpenLog-eagle-import:220KOHM-0402T-1/16W-1% -> SparkFun-Resistor:100k_0402; PROD_ID RES-15094 -> RES-25013
- SW3: renamed from S3; value RESET -> SMD_4.6x2.8mm_h2.5mm; footprint SparkFun_Artemis_OpenLog:TACTILE_SWITCH_SMD_4.6X2.8MM -> SparkFun-Switch:Push_SMD_4.6x2.8mm_h2.5mm; symbol SparkFun_Artemis_OpenLog-eagle-import:MOMENTARY-SWITCH-SPST-SMD-4.6X2.8MM -> SparkFun-Switch:SPST_Push_SMD_4.6x2.8mm_h2.5mm; PROD_ID SWCH-13065 -> SWCH-15606
- TP0: renamed from SCL0; value TEST-POINTTP_15TH_THRU -> 0.75mm; footprint SparkFun_Artemis_OpenLog:TP_15TH -> SparkFun-Connector:TestPoint-0.75mm; symbol SparkFun_Artemis_OpenLog-eagle-import:TEST-POINTTP_15TH_THRU -> SparkFun-Connector:TestPoint_0.75mm
- TP2: renamed from QWIIC_3.3V0; value TEST-POINTTP_15TH_THRU -> 0.75mm; footprint SparkFun_Artemis_OpenLog:TP_15TH -> SparkFun-Connector:TestPoint-0.75mm; symbol SparkFun_Artemis_OpenLog-eagle-import:TEST-POINTTP_15TH_THRU -> SparkFun-Connector:TestPoint_0.75mm
- TP3: renamed from GND0; value TEST-POINTTP_15TH_THRU -> 0.75mm; footprint SparkFun_Artemis_OpenLog:TP_15TH -> SparkFun-Connector:TestPoint-0.75mm; symbol SparkFun_Artemis_OpenLog-eagle-import:TEST-POINTTP_15TH_THRU -> SparkFun-Connector:TestPoint_0.75mm
- TP4: renamed from SDA0; value TEST-POINTTP_15TH_THRU -> 0.75mm; footprint SparkFun_Artemis_OpenLog:TP_15TH -> SparkFun-Connector:TestPoint-0.75mm; symbol SparkFun_Artemis_OpenLog-eagle-import:TEST-POINTTP_15TH_THRU -> SparkFun-Connector:TestPoint_0.75mm
- U4: value 3.3V -> AP2112K-3.3; footprint SparkFun_Artemis_OpenLog:SOT23-5 -> SparkFun-Semiconductor-Standard:SOT23-5; symbol SparkFun_Artemis_OpenLog-eagle-import:V_REG_AP2112K-3.3V -> SparkFun-Regulator:AP2112K-3.3; IMax (none) -> 600mA; Iq (none) -> 55µA; VMax (none) -> 6V
Connections:
- net 3.3V: now also D6.2 (A); no longer D6.A
- net 5V: now also D1.1 (K); no longer D1.C
- net ARTEMIS_~{RESET}: now also SW3.2; no longer SW3.3 (2), SW3.4 (2)
- net GND: now also TP3.1; no longer SW3.2 (1), TP3.P$1 (1)
- net QWIIC_3.3V: now also TP2.1; no longer TP2.P$1 (1)
- net RTC_BAT+: now also D3.2 (A); no longer D3.A
- net SCL: now also TP0.1; no longer TP0.P$1 (1)
- net SDA: now also TP4.1; no longer TP4.P$1 (1)
- net VCC_1: now also D3.1 (K), D6.1 (K); no longer D3.C, D6.C
- net V_BATT: now also D1.2 (A); no longer D1.A
Other:
- moved on the sheet: D11, D12, D2, R24, R25, R5, SW3, TP0, TP2, TP3, TP4, Y3

Commit message: Save point
Parts:
- JP0: renamed from VE0; value JUMPER-SMT_2_NO_SILK -> (none); footprint SparkFun_Artemis_OpenLog:SMT-JUMPER_2_NO_SILK -> SparkFun-Jumper:Jumper_2_NO; symbol SparkFun_Artemis_OpenLog-eagle-import:JUMPER-SMT_2_NO_SILK -> SparkFun-Jumper:SolderJumper_2_Open
Other:
- moved on the sheet: C10, C11, C2, C31, C32, C33, C5, C6, C7, C8, R6

Commit message: Save point (near the end)
Parts:
- removed FRAME1: FRAME-LEDGER, SparkFun_Artemis_OpenLog:CREATIVE_COMMONS, symbol SparkFun_Artemis_OpenLog-eagle-import:FRAME-LEDGER
- removed LOGO3: SPECIAL_INSTRUCTIONS-ORDERING, SparkFun_Artemis_OpenLog:ORDERING_INSTRUCTIONS, symbol SparkFun_Artemis_OpenLog-eagle-import:SPECIAL_INSTRUCTIONS-ORDERING
- FID1: renamed from FD1; value FIDUCIAL1X2 -> Fiducial_0.5mm; footprint SparkFun_Artemis_OpenLog:FIDUCIAL-1X2 -> SparkFun-Aesthetic:Fiducial_0.5mm_Mask1mm; symbol SparkFun_Artemis_OpenLog-eagle-import:FIDUCIAL1X2 -> SparkFun-Aesthetic:Fiducial_0.5mm
- FID2: renamed from FD2; value FIDUCIAL1X2 -> Fiducial_0.5mm; footprint SparkFun_Artemis_OpenLog:FIDUCIAL-1X2 -> SparkFun-Aesthetic:Fiducial_0.5mm_Mask1mm; symbol SparkFun_Artemis_OpenLog-eagle-import:FIDUCIAL1X2 -> SparkFun-Aesthetic:Fiducial_0.5mm
- FID3: renamed from FD3; value FIDUCIAL1X2 -> Fiducial_0.5mm; footprint SparkFun_Artemis_OpenLog:FIDUCIAL-1X2 -> SparkFun-Aesthetic:Fiducial_0.5mm_Mask1mm; symbol SparkFun_Artemis_OpenLog-eagle-import:FIDUCIAL1X2 -> SparkFun-Aesthetic:Fiducial_0.5mm
- FID4: renamed from FD4; value FIDUCIAL1X2 -> Fiducial_0.5mm; footprint SparkFun_Artemis_OpenLog:FIDUCIAL-1X2 -> SparkFun-Aesthetic:Fiducial_0.5mm_Mask1mm; symbol SparkFun_Artemis_OpenLog-eagle-import:FIDUCIAL1X2 -> SparkFun-Aesthetic:Fiducial_0.5mm
- ST1: renamed from H1; value STAND-OFF -> Standoff; footprint SparkFun_Artemis_OpenLog:STAND-OFF -> SparkFun-Hardware:Standoff; symbol SparkFun_Artemis_OpenLog-eagle-import:STAND-OFF -> SparkFun-Hardware:Standoff
- ST2: renamed from H2; value STAND-OFF -> Standoff; footprint SparkFun_Artemis_OpenLog:STAND-OFF -> SparkFun-Hardware:Standoff; symbol SparkFun_Artemis_OpenLog-eagle-import:STAND-OFF -> SparkFun-Hardware:Standoff
- ST3: renamed from H3; value STAND-OFF -> Standoff; footprint SparkFun_Artemis_OpenLog:STAND-OFF -> SparkFun-Hardware:Standoff; symbol SparkFun_Artemis_OpenLog-eagle-import:STAND-OFF -> SparkFun-Hardware:Standoff
- ST4: renamed from H4; value STAND-OFF -> Standoff; footprint SparkFun_Artemis_OpenLog:STAND-OFF -> SparkFun-Hardware:Standoff; symbol SparkFun_Artemis_OpenLog-eagle-import:STAND-OFF -> SparkFun-Hardware:Standoff
- U5: footprint SparkFun_Artemis_OpenLog:LGA-28 -> SparkFun-Semiconductor-Standard:LGA-28_5.2x3.8mm_P0.5mm; symbol SparkFun_Artemis_OpenLog-eagle-import:BNO086 -> SparkFun-Sensor:BNO086
- U8: value ARTEMIS_MODULE -> Artemis Module; footprint SparkFun_Artemis_OpenLog:ARTEMIS_FP -> SparkFun-Semiconductor-Nonstandard:Artemis_Module; symbol SparkFun_Artemis_OpenLog-eagle-import:ARTEMIS_MODULESMD -> SparkFun-IC-Microcontroller:Aretmis_Module
Connections:
- net ARTEMIS_~{RTS}: now also U10.4 (~{RTS}); no longer U10.5 (~{CTS})
Other:
- note added: "IMU - BNO086"
- note removed: "N. Seidle"
- note removed: "v10"
- company: (none) -> SparkFun Electronics
- title: (none) -> OpenLog Artemis
- moved on the sheet: BT1, C1, C10, C11, C2, C3, C4, C42, C43, C44, C46, C5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

Commit message: Save point
Parts:
- removed LOGO1: SFE_LOGO_NAME.1_INCH, SparkFun_Artemis_OpenLog:SFE_LOGO_NAME_.1, symbol SparkFun_Artemis_OpenLog-eagle-import:SFE_LOGO_NAME.1_INCH
- removed LOGO2: OSHW-LOGOS, SparkFun_Artemis_OpenLog:OSHW-LOGO-S, symbol SparkFun_Artemis_OpenLog-eagle-import:OSHW-LOGOS
- removed LOGO4, LOGO5: SFE_LOGO_FLAME.1_INCH, SparkFun_Artemis_OpenLog:SFE_LOGO_FLAME_.1, symbol SparkFun_Artemis_OpenLog-eagle-import:SFE_LOGO_FLAME.1_INCH
- added G1: OSHW_Logo, SparkFun-Aesthetic:Creative_Commons_License, symbol SparkFun-Aesthetic:OSHW_Logo
- added G2: SparkFun_Logo, symbol SparkFun-Aesthetic:SparkFun_Logo
- TP1: value TEST-POINT3 -> 1.0mm; footprint SparkFun_Artemis_OpenLog:PAD.03X.03 -> SparkFun-Connector:TestPoint-1.0mm; symbol SparkFun_Artemis_OpenLog-eagle-import:TEST-POINT3 -> SparkFun-Connector:TestPoint_1.0mm
Connections:
- net RTC_BAT+: now also TP1.1; no longer TP1.P$1 (1)
- new net: U5.1 (RESV_NC), U5.12 (RESV_NC), U5.13 (RESV_NC), U5.21 (RESV_NC), U5.22 (RESV_NC), U5.23 (RESV_NC), U5.24 (RESV_NC), U5.7 (RESV_NC), U5.8 (RESV_NC)
Other:
- moved on the sheet: TP1

Commit message: Updates microSD - save point
Parts:
- J6: value MICRO-SD -> microSD; footprint SparkFun_Artemis_OpenLog:MICRO-SD-SOCKET -> SparkFun-Connector:microSD_SOCKET; symbol SparkFun_Artemis_OpenLog-eagle-import:MICRO-SD-SDIOPUSH-PUSH -> SparkFun-Connector:microSD_PushPush_No_Drill
Connections:
- net DAT1: now also J6.8 (DAT1); no longer J6.DAT1 (DAT1/NC)
- net DAT2: now also J6.1 (DAT2); no longer J6.DAT2 (DAT2/NC)
- net GND: now also J6.10 (GND), J6.11 (CD), J6.12 (CD), J6.6 (GND), J6.9 (SHIELD); no longer J6.CD1 (SHIELD), J6.GND, J6.GND1 (GND), J6.GND3 (GND)
- net MICROSD_~{CS}: now also J6.2 (DAT3/CD); no longer J6.CS/DAT3 (DAT3/~{CS})
- net SCK: now also J6.5 (CLK/SCK); no longer J6.SCLK (CLK/SCK)
- net SDI: now also J6.7 (DAT0/SDO); no longer J6.DO/DAT0 (DAT0/SDO)
- net SDO: now also J6.3 (CMD/SDI); no longer J6.DI/CMD (CMD/SDI)
- net at C46.1, Q2.3 (D): now also J6.4 (VDD); no longer J6.VCC
Other:
- note removed: "Linear 3.3V"
- moved on the sheet: C2, J3, R2, R6, R7

Commit message: All KiCad components - save point
Parts:
- U1: value 3.0V Supervisor -> MAX810TTRG; footprint SparkFun_Artemis_OpenLog:SOT23-3 -> SparkFun-Semiconductor-Standard:SOT23-3; symbol SparkFun_Artemis_OpenLog-eagle-import:V_SUPERVISOR -> SparkFun-IC-Power:MAX810TTRG
- Y1, Y3: footprint SparkFun_Artemis_OpenLog:CRYSTAL-SMD-3.2X1.5MM -> SparkFun-Clock:Crystal_SMD_3.2x1.5mm; symbol SparkFun_Artemis_OpenLog-eagle-import:CRYSTAL-32.768KHZSMD-3.2X1.5 -> SparkFun-Clock:Crystal_32.768kHz_3.2x1.5mm; PROD_ID XTAL-13062 -> XTAL-25022
Connections:
- net at C6.1, U5.26 (CLKSEL1): now also Y1.1; no longer Y1.P$1 (1)
- net at C8.1, U5.27 (XIN32): now also Y1.2; no longer Y1.P$2 (2)
- net at C30.2, U8.XI: now also Y3.1; no longer Y3.P$1 (1)
- net at C29.2, U8.XO: now also Y3.2; no longer Y3.P$2 (2)
Changed lines of the file:
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@@
 	(wire
 		(pts
-			(xy 72.39 143.51) (xy 69.85 143.51)
-		)
-		(stroke
-			(width 0.1524)
-			(type solid)
-		)
-	)
-	(wire
-		(pts
 			(xy 76.2 287.02) (xy 78.74 287.02)
 		)
@@
 	(wire
 		(pts
-			(xy 69.85 148.59) (xy 69.85 151.13)
-		)
-		(stroke
-			(width 0.1524)
-			(type solid)
-		)
-	)
-	(wire
-		(pts
 			(xy 264.16 55.88) (xy 264.16 60.96)
 		)
@@
 	(wire
 		(pts
-			(xy 69.85 140.97) (xy 69.85 143.51)
+			(xy 81.28 134.62) (xy 81.28 135.89)
 		)
 		(stroke
@@
 	(wire
 		(pts
+			(xy 81.28 156.21) (xy 81.28 157.48)
+		)
+		(stroke
+			(width 0)
+			(type default)
+		)
+	)
+	(wire
+		(pts
 			(xy 320.04 218.44) (xy 320.04 220.98)
 		)
@@
 	(wire
 		(pts
-			(xy 72.39 148.59) (xy 69.85 148.59)
-		)
-		(stroke
-			(width 0.1524)
-			(type solid)
-		)
-	)
-	(wire
-		(pts
 			(xy 207.01 58.42) (xy 207.01 66.04)
 		)
@@
 	(symbol
 		(lib_id "SparkFun-PowerSymbol:GND")
-		(at 69.85 151.13 0)
+		(at 81.28 157.48 0)
 		(unit 1)
 		(body_style 1)
@@
 		(dnp no)
 		(property "Reference" "#PWR8"
-			(at 69.85 157.48 0)
+			(at 81.28 163.83 0)
 			(hide yes)
 			(show_name no)
@@
 		)
 		(property "Value" "GND"
-			(at 69.85 154.94 0)
+			(at 81.28 161.29 0)
 			(show_name no)
 			(do_not_autoplace yes)
@@
 		)
 		(property "Footprint" ""
-			(at 69.85 151.13 0)
+			(at 81.28 157.48 0)
 			(hide yes)
 			(show_name no)
@@
 		)
 		(property "Datasheet" ""
-			(at 69.85 151.13 0)
+			(at 81.28 157.48 0)
 			(hide yes)
 			(show_name no)
@@
 		)
 		(property "Description" "Power symbol creates a global label with name \"GND\" , ground"
-			(at 69.85 160.02 0)
+			(at 81.28 166.37 0)
 			(hide yes)
 			(show_name no)
@@
 	)
 	(symbol
-		(lib_id "SparkFun_Artemis_OpenLog-eagle-import:CRYSTAL-32.768KHZSMD-3.2X1.5")
+		(lib_id "SparkFun-Clock:Crystal_32.768kHz_3.2x1.5mm")
 		(at 304.8 250.19 90)
 		(unit 1)
@@
 		(dnp no)
 		(property "Reference" "Y1"
-			(at 308.356 249.682 90)
+			(at 302.26 250.19 0)
 			(show_name no)
 			(do_not_autoplace no)
 			(effects
 				(font
-					(size 1.778 1.5113)
+					(size 1.27 1.27)
 				)
-				(justify top)
 			)
 		)
 		(property "Value" "32.768kHz"
-			(at 310.388 253.238 90)
+			(at 307.34 250.19 0)
 			(show_name no)
 			(do_not_autoplace no)
 			(effects
 				(font
-					(size 1.27 1.0795)
+					(size 1.27 1.27)
 				)
-				(justify top)
 			)
 		)
-		(property "Footprint" "SparkFun_Artemis_OpenLog:CRYSTAL-SMD-3.2X1.5MM"
-			(at 304.8 250.19 0)
+		(property "Footprint" "SparkFun-Clock:Crystal_SMD_3.2x1.5mm"
+			(at 312.42 250.19 0)
 			(hide yes)
 			(show_name no)
@@
 			)
 		)
-		(property "Datasheet" ""
-			(at 304.8 250.19 0)
+		(property "Datasheet" "https://abracon.com/Resonators/ABS07.pdf"
+			(at 309.88 250.19 0)
 			(hide yes)
 			(show_name no)
@@
 			)
 		)
-		(property "Description" ""
-			(at 304.8 250.19 0)
+		(property "Description" "Crystal"
+			(at 317.5 250.19 0)
 			(hide yes)
 			(show_name no)
@@
 			)
 		)
-		(property "PROD_ID" "XTAL-13062"
-			(at 304.8 255.27 0)
+		(property "PROD_ID" "XTAL-25022"
+			(at 314.96 250.19 0)
 			(hide yes)
 			(show_name no)
@@
 			)
 		)
-		(pin "P$1"
+		(pin "1"
 		)
-		(pin "P$2"
+		(pin "2"
 		)
 		(instances
@@
 	)
 	(symbol
-		(lib_id "SparkFun_Artemis_OpenLog-eagle-import:V_SUPERVISOR")
-		(at 80.01 146.05 0)
+		(lib_id "SparkFun-IC-Power:MAX810TTRG")
+		(at 81.28 146.05 0)
 		(unit 1)
 		(body_style 1)
@@
 		(dnp no)
 		(property "Reference" "U1"
-			(at 74.93 140.462 0)
+			(at 82.804 138.176 0)
 			(show_name no)
 			(do_not_autoplace no)
 			(effects
 				(font
-					(size 1.778 1.5113)
+					(size 1.27 1.27)
 				)
 				(justify left bottom)
 			)
 		)
-		(property "Value" "3.0V Supervisor"
-			(at 74.93 153.67 0)
+		(property "Value" "MAX810TTRG"
+			(at 82.804 155.448 0)
 			(show_name no)
 			(do_not_autoplace no)
 			(effects
 				(font
-					(size 1.778 1.5113)
+					(size 1.27 1.27)
 				)
 				(justify left bottom)
 			)
 		)
-		(property "Footprint" "SparkFun_Artemis_OpenLog:SOT23-3"
-			(at 80.01 146.05 0)
+		(property "Footprint" "SparkFun-Semiconductor-Standard:SOT23-3"
+			(at 81.788 179.578 0)
 			(hide yes)
 			(show_name no)
@@
 			)
 		)
-		(property "Datasheet" ""
-			(at 80.01 146.05 0)
+		(property "Datasheet" "https://www.farnell.com/datasheets/89200.pdf"
+			(at 80.264 170.434 0)
 			(hide yes)
 			(show_name no)
@@
 			)
 		)
-		(property "Description" ""
-			(at 80.01 146.05 0)
+		(property "Description" "The MAX809 and MAX810 are cost−effective system supervisor circuits designed to monitor VCC in digital systems and provide a reset signal to the host processor when necessary. No external components are required."
+			(at 82.042 167.64 0)
 			(hide yes)
 			(show_name no)
@@
 		)
 		(property "PROD_ID" "IC-14809"
-			(at 80.01 156.718 0)
+			(at 81.28 177.8 0)
 			(hide yes)
 			(show_name no)
@@
 	(symbol
 		(lib_id "SparkFun_Artemis_OpenLog-eagle-import:3.3V")
-		(at 69.85 140.97 0)
+		(at 81.28 134.62 0)
 		(unit 1)
 		(body_style 1)
@@
 		(dnp no)
 		(property "Reference" "#SUPPLY4"
-			(at 69.85 140.97 0)
+			(at 81.28 134.62 0)
 			(hide yes)
 			(show_name no)
@@
 		)
 		(property "Value" "3.3V"
-			(at 69.85 138.176 0)
+			(at 81.28 131.826 0)
 			(show_name no)
 			(do_not_autoplace no)
@@
 		)
 		(property "Footprint" ""
-			(at 69.85 140.97 0)
+			(at 81.28 134.62 0)
 			(hide yes)
 			(show_name no)
@@
 		)
 		(property "Datasheet" ""
-			(at 69.85 140.97 0)
+			(at 81.28 134.62 0)
 			(hide yes)
 			(show_name no)
@@
 		)
 		(property "Description" ""
-			(at 69.85 140.97 0)
+			(at 81.28 134.62 0)
 			(hide yes)
 			(show_name no)
@@
 	)
 	(symbol
-		(lib_id "SparkFun_Artemis_OpenLog-eagle-import:CRYSTAL-32.768KHZSMD-3.2X1.5")
+		(lib_id "SparkFun-Clock:Crystal_32.768kHz_3.2x1.5mm")
 		(at 55.88 245.11 270)
 		(unit 1)
@@
 		(dnp no)
 		(property "Reference" "Y3"
-			(at 55.88 241.554 90)
+			(at 58.42 245.11 0)
 			(show_name no)
 			(do_not_autoplace no)
 			(effects
 				(font
-					(size 1.778 1.5113)
+					(size 1.27 1.27)
 				)
-				(justify bottom)
 			)
 		)
 		(property "Value" "32.768kHz"
-			(at 65.532 244.602 90)
+			(at 53.34 245.11 0)
 			(show_name no)
 			(do_not_autoplace no)
 			(effects
 				(font
-					(size 1.778 1.5113)
+					(size 1.27 1.27)
 				)
-				(justify bottom)
 			)
 		)
-		(property "Footprint" "SparkFun_Artemis_OpenLog:CRYSTAL-SMD-3.2X1.5MM"
-			(at 55.88 245.11 0)
+		(property "Footprint" "SparkFun-Clock:Crystal_SMD_3.2x1.5mm"
+			(at 48.26 245.11 0)
 			(hide yes)
 			(show_name no)
@@
 			)
 		)
-		(property "Datasheet" ""
-			(at 55.88 245.11 0)
+		(property "Datasheet" "https://abracon.com/Resonators/ABS07.pdf"
+			(at 50.8 245.11 0)
 			(hide yes)
 			(show_name no)
@@
 			)
 		)
-		(property "Description" ""
-			(at 55.88 245.11 0)
+		(property "Description" "Crystal"
+			(at 43.18 245.11 0)
 			(hide yes)
 			(show_name no)
@@
 			)
 		)
-		(property "PROD_ID" "XTAL-13062"
-			(at 55.88 250.19 0)
+		(property "PROD_ID" "XTAL-25022"
+			(at 45.72 245.11 0)
 			(hide yes)
 			(show_name no)
@@
 			)
 		)
-		(pin "P$1"
+		(pin "2"
 		)
-		(pin "P$2"
+		(pin "1"
 		)
 		(instances

Commit message: Updates design with silk
Other:
- note added: "LiPo Charger - MCP73831"
- note added: "RTC Battery and Battery Supervisor"
- note added: "USB-to-Serial Converter - CH340E"
- note added: "microSD"
- note removed: "LiPo Charger"
- note removed: "RTC Battery"
- note removed: "USB-to-Serial Converter"
- note removed: "μSD"
- moved on the sheet: C40, C41, D11, D12, J8, R24, R25, R26, R27, R8, U10

Commit message: Updates the 5V symbol
Parts:
- renumbered C32 to C1, C3 to C10, C10 to C11, C1 to C12, C43 to C13, C2 to C14, C42 to C15, C44 to C16, C9 to C17, C6 to C18, C8 to C19, C33 to C2, C46 to C20, C7 to C21, C5 to C22, C31 to C3, C30 to C4, C29 to C5, C41 to C6, C40 to C7, C4 to C8, C11 to C9, D6 to D1, D3 to D2, D12 to D3, D11 to D4, D1 to D5, D2 to D6, D20 to D7, D9 to D8, FID3 to FID2, FID2 to FID3, G2 to G1, G1 to G2, J8 to J1, J4 to J2, J14 to J3, J7 to J4, J2 to J6, J3 to J7, J11 to J8, J6 to J9, JP0 to JP1, Q2 to Q1, R29 to R10, R2 to R11, R28 to R12, R9 to R13, R10 to R14, R7 to R15, R6 to R16, R11 to R17, R3 to R18, R22 to R19, R8 to R2, R23 to R20, R26 to R3, R27 to R4, R25 to R5, R24 to R6, R4 to R7, R5 to R8, R12 to R9, ST3 to ST2, ST2 to ST3, SW3 to SW1, TP0 to TP2, TP4 to TP3, TP2 to TP4, TP3 to TP5, U10 to U2, U8 to U3, U2 to U4, U3 to U5, U5 to U6, U4 to U7, Y3 to Y1, Y1 to Y2
