File: Hardware/SparkFun_Artemis_OpenLog/SparkFun_Artemis_OpenLog.kicad_sch (KiCad schematic)
At the start: 88 parts, among them J1 USB_C_Receptacle, J2 Conn_01x06, J3 SWD, J4 Conn_01x01, J5 JST_2mm_LiPo, J6 Conn_01x02, J7 Conn_01x02, J8 Qwiic_RA, J9 microSD, Q1 DMG2305UX, SW1 SMD_4.6x2.8mm_h2.5mm, U1 MAX810TTRG, U2 CH340E, U3 Artemis Module, U4 MCP73831, U5 AP2112K-3.3, U6 BNO086, U7 AP2112K-3.3, Y1 32.768kHz, Y2 32.768kHz

Commit message: Updates power symbols for VBATT, 3.3V, and VCC
Connections:
- net VCC_1: no longer C1.1, C2.1, C3.2, R12.2, U3.VDD@36 (VDD*2), U3.VDD@37 (VDD*2)
- new net VCC: C1.1, C2.1, C3.2, R12.2, U3.VDD@36 (VDD*2), U3.VDD@37 (VDD*2)

Commit message: Fixes the many DRC issues
Connections:
- net VCC_1 is gone; now on net VCC: D1.1 (K), D2.1 (K), R1.2
Other:
- moved on the sheet: R13
Changed lines of the file:
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@@
 	(text "300uA Leakage"
 		(exclude_from_sim no)
-		(at 54.61 151.13 90)
+		(at 69.85 147.32 0)
 		(effects
 			(font
 				(size 1.27 1.27)
 			)
-			(justify left bottom)
+			(justify right bottom)
 		)
 	)
 	(text "0.65uA Leakage\n0.3V drop at 10mA"
 		(exclude_from_sim no)
-		(at 31.242 147.32 90)
+		(at 16.51 127 0)
 		(effects
 			(font
@@
 	(text "1mAhr Capacity"
 		(exclude_from_sim no)
-		(at 46.99 163.83 0)
+		(at 41.91 163.83 0)
 		(effects
 			(font
@@
 	(text "LiPo Range: 3.6-4.2V"
 		(exclude_from_sim no)
-		(at 165.1 25.4 0)
+		(at 157.48 33.02 0)
 		(effects
 			(font
@@
 	(wire
 		(pts
-			(xy 299.72 217.17) (xy 299.72 219.71)
+			(xy 299.72 218.44) (xy 299.72 219.71)
 		)
 		(stroke
@@
 	(wire
 		(pts
-			(xy 299.72 208.28) (xy 299.72 212.09)
-		)
-		(stroke
-			(width 0.1524)
-			(type solid)
-		)
-	)
-	(wire
-		(pts
 			(xy 73.66 248.92) (xy 73.66 243.84)
 		)
@@
 	(wire
 		(pts
+			(xy 299.72 213.36) (xy 299.72 212.09)
+		)
+		(stroke
+			(width 0)
+			(type default)
+		)
+	)
+	(wire
+		(pts
 			(xy 256.54 222.25) (xy 256.54 219.71)
 		)
@@
 	(wire
 		(pts
-			(xy 312.42 210.82) (xy 312.42 213.36)
+			(xy 312.42 212.09) (xy 312.42 213.36)
 		)
 		(stroke
@@
 	(wire
 		(pts
-			(xy 320.04 210.82) (xy 320.04 213.36)
+			(xy 320.04 212.09) (xy 320.04 213.36)
 		)
 		(stroke
@@
 	(wire
 		(pts
-			(xy 320.04 208.28) (xy 320.04 210.82)
-		)
-		(stroke
-			(width 0.1524)
-			(type solid)
-		)
-	)
-	(wire
-		(pts
 			(xy 78.74 236.22) (xy 77.47 236.22)
 		)
@@
 	(wire
 		(pts
-			(xy 312.42 208.28) (xy 312.42 210.82)
-		)
-		(stroke
-			(width 0.1524)
-			(type solid)
-		)
-	)
-	(wire
-		(pts
 			(xy 160.02 167.64) (xy 162.56 167.64)
 		)
@@
 		(dnp no)
 		(property "Reference" "D1"
-			(at 36.83 133.35 0)
+			(at 34.29 129.54 90)
 			(show_name no)
 			(do_not_autoplace no)
@@
 		)
 		(property "Value" "BAT20J"
-			(at 43.18 133.35 0)
+			(at 34.29 132.08 90)
 			(show_name no)
 			(do_not_autoplace no)
@@
 		)
 		(property "IMax" "1A"
-			(at 45.72 133.35 0)
+			(at 34.29 134.62 90)
 			(show_name no)
 			(do_not_autoplace no)
@@
 		)
 		(property "VForward" "0.62V"
-			(at 48.26 133.35 0)
+			(at 34.29 137.16 90)
 			(show_name no)
 			(do_not_autoplace no)
@@
 		)
 		(property "VReverse" "23V"
-			(at 50.8 133.35 0)
+			(at 34.29 139.7 90)
 			(show_name no)
 			(do_not_autoplace no)
@@
 	(symbol
 		(lib_id "SparkFun-Resistor:100k_0402")
-		(at 299.72 214.63 90)
+		(at 299.72 215.9 90)
 		(unit 1)
 		(body_style 1)
@@
 		(dnp no)
 		(property "Reference" "R13"
-			(at 302.26 214.63 0)
+			(at 302.26 215.9 0)
 			(show_name no)
 			(do_not_autoplace no)
@@
 		)
 		(property "Value" "100k"
-			(at 297.18 214.63 0)
+			(at 297.18 215.9 0)
 			(show_name no)
 			(do_not_autoplace no)
@@
 		)
 		(property "Footprint" "SparkFun-Resistor:R_0402_1005Metric"
-			(at 304.038 214.63 0)
+			(at 304.038 215.9 0)
 			(hide yes)
 			(show_name no)
@@
 		)
 		(property "Datasheet" "https://www.vishay.com/docs/20035/dcrcwe3.pdf"
-			(at 308.61 214.63 0)
+			(at 308.61 215.9 0)
 			(hide yes)
 			(show_name no)
@@
 		)
 		(property "Description" "Resistor"
-			(at 311.15 214.63 0)
+			(at 311.15 215.9 0)
 			(hide yes)
 			(show_name no)
@@
 		)
 		(property "PROD_ID" "RES-25013"
-			(at 306.07 214.63 0)
+			(at 306.07 215.9 0)
 			(hide yes)
 			(show_name no)
@@
 	(symbol
 		(lib_id "SparkFun-PowerSymbol:3.3V")
-		(at 299.72 208.28 0)
+		(at 299.72 212.09 0)
 		(unit 1)
 		(body_style 1)
@@
 		(dnp no)
 		(property "Reference" "#PWR20"
-			(at 299.72 212.09 0)
+			(at 299.72 215.9 0)
 			(hide yes)
 			(show_name no)
@@
 		)
 		(property "Value" "3.3V"
-			(at 299.72 204.47 0)
+			(at 299.72 208.28 0)
 			(show_name no)
 			(do_not_autoplace yes)
@@
 		)
 		(property "Footprint" ""
-			(at 299.72 208.28 0)
+			(at 299.72 212.09 0)
 			(hide yes)
 			(show_name no)
@@
 		)
 		(property "Datasheet" ""
-			(at 299.72 208.28 0)
+			(at 299.72 212.09 0)
 			(hide yes)
 			(show_name no)
@@
 		)
 		(property "Description" "Power symbol creates a global label with name \"3.3V\""
-			(at 299.72 214.63 0)
+			(at 299.72 218.44 0)
 			(hide yes)
 			(show_name no)
@@
 		(dnp no)
 		(property "Reference" "D2"
-			(at 44.196 148.844 0)
+			(at 50.8 140.97 90)
 			(show_name no)
 			(do_not_autoplace no)
@@
 		)
 		(property "Value" "BAT60A"
-			(at 44.196 143.51 0)
+			(at 50.8 143.51 90)
 			(show_name no)
 			(do_not_autoplace no)
@@
 		)
 		(property "IMax" "3A"
-			(at 49.53 139.7 0)
+			(at 50.8 146.05 90)
 			(show_name no)
 			(do_not_autoplace no)
@@
 		)
 		(property "VDrop" "0.28V"
-			(at 49.53 144.526 0)
+			(at 50.8 148.59 90)
 			(show_name no)
 			(do_not_autoplace no)
@@
 		)
 		(property "VMax" "10V"
-			(at 49.53 149.606 0)
+			(at 50.8 151.13 90)
 			(show_name no)
 			(do_not_autoplace no)
@@
 			)
 		)
-		(property "Value" "VCC_1"
+		(property "Value" "VCC"
 			(at 46.99 124.46 0)
 			(show_name no)
@@
 	(symbol
 		(lib_id "SparkFun-PowerSymbol:3.3V")
-		(at 312.42 208.28 0)
+		(at 312.42 212.09 0)
 		(unit 1)
 		(body_style 1)
@@
 		(dnp no)
 		(property "Reference" "#PWR21"
-			(at 312.42 212.09 0)
+			(at 312.42 215.9 0)
 			(hide yes)
 			(show_name no)
@@
 		)
 		(property "Value" "3.3V"
-			(at 312.42 204.47 0)
+			(at 312.42 208.28 0)
 			(show_name no)
 			(do_not_autoplace yes)
@@
 		)
 		(property "Footprint" ""
-			(at 312.42 208.28 0)
+			(at 312.42 212.09 0)
 			(hide yes)
 			(show_name no)
@@
 		)
 		(property "Datasheet" ""
-			(at 312.42 208.28 0)
+			(at 312.42 212.09 0)
 			(hide yes)
 			(show_name no)
@@
 		)
 		(property "Description" "Power symbol creates a global label with name \"3.3V\""
-			(at 312.42 214.63 0)
+			(at 312.42 218.44 0)
 			(hide yes)
 			(show_name no)
@@
 	(symbol
 		(lib_id "SparkFun-PowerSymbol:3.3V")
-		(at 320.04 208.28 0)
+		(at 320.04 212.09 0)
 		(unit 1)
 		(body_style 1)
@@
 		(dnp no)
 		(property "Reference" "#PWR22"
-			(at 320.04 212.09 0)
+			(at 320.04 215.9 0)
 			(hide yes)
 			(show_name no)
@@
 		)
 		(property "Value" "3.3V"
-			(at 320.04 204.47 0)
+			(at 320.04 208.28 0)
 			(show_name no)
 			(do_not_autoplace yes)
@@
 		)
 		(property "Footprint" ""
-			(at 320.04 208.28 0)
+			(at 320.04 212.09 0)
 			(hide yes)
 			(show_name no)
@@
 		)
 		(property "Datasheet" ""
-			(at 320.04 208.28 0)
+			(at 320.04 212.09 0)
 			(hide yes)
 			(show_name no)
@@
 		)
 		(property "Description" "Power symbol creates a global label with name \"3.3V\""
-			(at 320.04 214.63 0)
+			(at 320.04 218.44 0)
 			(hide yes)
 			(show_name no)
@@
 		(dnp no)
 		(property "Reference" "R1"
-			(at 36.576 147.828 0)
+			(at 36.576 147.828 90)
 			(show_name no)
 			(do_not_autoplace no)
@@
 		)
 		(property "Value" "2.2k"
-			(at 36.576 143.764 0)
+			(at 35.56 149.86 90)
 			(show_name no)
 			(do_not_autoplace no)

Commit message: Updated resistor values
Parts:
- JP1: value (none) -> VE
- R15: value 200k -> 2M; footprint SparkFun-Resistor:R_0402_1005Metric -> SparkFun-Resistor:R_0603_1608Metric; symbol SparkFun-Resistor:200k_0402 -> SparkFun-Resistor:2M_0603; PROD_ID RES-15347 -> RES-15186
- R16: value 100k -> 1M; footprint SparkFun-Resistor:R_0402_1005Metric -> SparkFun-Resistor:R_0603_1608Metric; symbol SparkFun-Resistor:100k_0402 -> SparkFun-Resistor:1M_0603; PROD_ID RES-25013 -> RES-07868
Changed lines of the file:
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@@
 	)
 	(symbol
-		(lib_id "SparkFun-Resistor:200k_0402")
+		(lib_id "SparkFun-Resistor:2M_0603")
 		(at 320.04 52.07 90)
 		(unit 1)
@@
 			)
 		)
-		(property "Value" "200k"
+		(property "Value" "2M"
 			(at 317.5 52.07 0)
 			(show_name no)
@@
 			)
 		)
-		(property "Footprint" "SparkFun-Resistor:R_0402_1005Metric"
+		(property "Footprint" "SparkFun-Resistor:R_0603_1608Metric"
 			(at 324.358 52.07 0)
 			(hide yes)
@@
 			)
 		)
-		(property "PROD_ID" "RES-15347"
+		(property "PROD_ID" "RES-15186"
 			(at 326.39 52.07 0)
 			(hide yes)
@@
 			)
 		)
-		(property "Value" ""
+		(property "Value" "VE"
 			(at 165.1 256.54 0)
 			(show_name no)
@@
 	)
 	(symbol
-		(lib_id "SparkFun-Resistor:100k_0402")
+		(lib_id "SparkFun-Resistor:1M_0603")
 		(at 320.04 60.96 90)
 		(unit 1)
@@
 			)
 		)
-		(property "Value" "100k"
+		(property "Value" "1M"
 			(at 317.5 60.96 0)
 			(show_name no)
@@
 			)
 		)
-		(property "Footprint" "SparkFun-Resistor:R_0402_1005Metric"
+		(property "Footprint" "SparkFun-Resistor:R_0603_1608Metric"
 			(at 324.358 60.96 0)
 			(hide yes)
@@
 			)
 		)
-		(property "PROD_ID" "RES-25013"
+		(property "PROD_ID" "RES-07868"
 			(at 326.39 60.96 0)
 			(hide yes)

Commit message: Save before switch for IMU update
Parts:
- added C23: 10uF, SparkFun-Capacitor:C_0402_1005Metric, symbol SparkFun-Capacitor:10uF_0402_6.3V_20%
- C20: value 0.1uF -> 10uF; symbol SparkFun-Capacitor:0.1uF_0402_16V_10% -> SparkFun-Capacitor:10uF_0402_6.3V_20%; PROD_ID CAP-25565 -> CAP-14848; Tolerance 10% -> 20%; Voltage 16V -> 6.3V
Connections:
- net 3.3V: now also C23.1
- net GND: now also C23.2
Other:
- moved on the sheet: C20, Q1

Commit message: Fixes BNO symbol, adds parts to mosfet
Parts:
- added Q2: DMG2305UX, SparkFun-Semiconductor-Standard:SOT23-3, symbol SparkFun-DiscreteSemi:Q_PMOS_4.2A_20V
- added R21, R22: 100k, SparkFun-Resistor:R_0402_1005Metric, symbol SparkFun-Resistor:100k_0402
Connections:
- net 3.3V: now also Q2.2 (S)
- net GND: now also R21.1, R22.1
- net ICM_PWR: now also Q2.1 (G), R22.2
- net MICROSD_PWR: now also R21.2
- net at C18.1, U6.26 (CLKSEL1/XOUT32): now also Y2.2; no longer Y2.1
- net at C19.1, U6.27 (XIN32): now also Y2.1; no longer Y2.2
- net ~{RST}: no longer names the net of R13.1, U6.11 (~{RST})
- new net 3.3V_P: Q2.3 (D)
Other:
- moved on the sheet: C11, C17, C18, C19, C9, R13, R14, R17, R9, Y2
