File: Hardware/SparkFun_Artemis_OpenLog/SparkFun_Artemis_OpenLog.kicad_pcb (KiCad board)
At the start: 4 copper layers, 30.5 x 30.5 mm, 92 parts, among them J11 Qwiic_RA, J14 SWD, J2 Conn_01x02, J3 Conn_01x02, J4 Conn_01x06, J5 JST_2mm_LiPo, J6 MICRO-SD, J7 Conn_01x01, J8 USB_C_Receptacle, Q2 DMG2305UX, SW3 SMD_4.6x2.8mm_h2.5mm, U1 3.0V Supervisor, U10 CH340E, U2 MCP73831, U3 AP2112K-3.3, U4 AP2112K-3.3, U5 BNO086, U8 ARTEMIS_MODULE, Y1 32.768kHz, Y3 32.768kHz

Commit message: Save point
Parts:
- removed VE0: JUMPER-SMT_2_NO_SILK, SMT-JUMPER_2_NO_SILK
- added JP0: ~, SparkFun-Jumper:Jumper_2_NO, F.Cu at (142.2, 108.8)
Changed lines of the file:
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@@
 		(embedded_fonts no)
 	)
+	(footprint "SparkFun-Jumper:Jumper_2_NO"
+		(layer "F.Cu")
+		(at 142.1511 108.8136 -90)
+		(tags "SparkFun")
+		(property "Reference" "JP0"
+			(at 0 -1.143 90)
+			(layer "F.Fab")
+			(effects
+				(font
+					(size 0.5 0.5)
+					(thickness 0.1)
+					(bold yes)
+				)
+				(justify top)
+			)
+		)
+		(property "Value" "~"
+			(at 0 1.143 90)
+			(layer "F.Fab")
+			(effects
+				(font
+					(size 0.5 0.5)
+					(thickness 0.1)
+					(bold yes)
+				)
+				(justify bottom)
+			)
+		)
+		(property "Datasheet" ""
+			(at 0 0 270)
+			(unlocked yes)
+			(layer "F.Fab")
+			(hide yes)
+			(effects
+				(font
+					(size 1.27 1.27)
+				)
+			)
+		)
+		(property "Description" "Solder Jumper, 2-pole, open"
+			(at 0 0 270)
+			(unlocked yes)
+			(layer "F.Fab")
+			(hide yes)
+			(effects
+				(font
+					(size 1.27 1.27)
+				)
+			)
+		)
+		(property ki_fp_filters "SolderJumper*Open*")
+		(sheetname "/")
+		(sheetfile "SparkFun_Artemis_OpenLog.kicad_sch")
+		(units
+			(unit
+				(name "A")
+				(pins "1" "2")
+			)
+		)
+		(duplicate_pad_numbers_are_jumpers no)
+		(fp_line
+			(start 0.8636 1.016)
+			(end -0.8636 1.016)
+			(stroke
+				(width 0.1524)
+				(type solid)
+			)
+			(layer "F.SilkS")
+		)
+		(fp_line
+			(start -1.1176 0.762)
+			(end -1.1176 -0.762)
+			(stroke
+				(width 0.1524)
+				(type solid)
+			)
+			(layer "F.SilkS")
+		)
+		(fp_line
+			(start 1.1176 0.762)
+			(end 1.1176 -0.762)
+			(stroke
+				(width 0.1524)
+				(type solid)
+			)
+			(layer "F.SilkS")
+		)
+		(fp_line
+			(start -0.8636 -1.016)
+			(end 0.8636 -1.016)
+			(stroke
+				(width 0.1524)
+				(type solid)
+			)
+			(layer "F.SilkS")
+		)
+		(fp_arc
+			(start -0.8636 1.016)
+			(mid -1.043205 0.941605)
+			(end -1.1176 0.762)
+			(stroke
+				(width 0.1524)
+				(type solid)
+			)
+			(layer "F.SilkS")
+		)
+		(fp_arc
+			(start 1.1176 0.762)
+			(mid 1.043205 0.941605)
+			(end 0.8636 1.016)
+			(stroke
+				(width 0.1524)
+				(type solid)
+			)
+			(layer "F.SilkS")
+		)
+		(fp_arc
+			(start -1.1176 -0.762)
+			(mid -1.043205 -0.941605)
+			(end -0.8636 -1.016)
+			(stroke
+				(width 0.1524)
+				(type solid)
+			)
+			(layer "F.SilkS")
+		)
+		(fp_arc
+			(start 0.8636 -1.016)
+			(mid 1.043205 -0.941605)
+			(end 1.1176 -0.762)
+			(stroke
+				(width 0.1524)
+				(type solid)
+			)
+			(layer "F.SilkS")
+		)
+		(fp_rect
+			(start 1 -0.9)
+			(end -1 0.9)
+			(stroke
+				(width 0.1)
+				(type default)
+			)
+			(fill no)
+			(layer "F.CrtYd")
+		)
+		(pad "1" smd rect
+			(at -0.4064 0 270)
+			(size 0.635 1.27)
+			(layers "F.Cu" "F.Mask")
+			(net "Net-(JP0-A)")
+			(pinfunction "A_1")
+			(pintype "passive")
+			(thermal_bridge_angle 0)
+		)
+		(pad "2" smd rect
+			(at 0.4064 0 270)
+			(size 0.635 1.27)
+			(layers "F.Cu" "F.Mask")
+			(net "VREG_EN")
+			(pinfunction "B_2")
+			(pintype "passive")
+			(thermal_bridge_angle 0)
+		)
+		(embedded_fonts no)
+	)
 	(footprint "SparkFun-Battery:ML414H_IV01E"
 		(layer "F.Cu")
@@
 		)
 	)
-	(footprint "SMT-JUMPER_2_NO_SILK"
-		(layer "F.Cu")
-		(at 142.1511 108.8136 -90)
-		(property "Reference" "VE0"
-			(at 0 -1.143 90)
-			(unlocked yes)
-			(layer "F.SilkS")
-			(effects
-				(font
-					(size 0.512064 0.512064)
-					(thickness 0.097536)
-				)
-				(justify top)
-			)
-		)
-		(property "Value" "JUMPER-SMT_2_NO_SILK"
-			(at 0 1.143 90)
-			(unlocked yes)
-			(layer "F.Fab")
-			(effects
-				(font
-					(size 0.512064 0.512064)
-					(thickness 0.097536)
-				)
-				(justify bottom)
-			)
-		)
-		(property "Datasheet" ""
-			(at 0 0 90)
-			(unlocked yes)
-			(layer "F.Fab")
-			(hide yes)
-			(effects
-				(font
-					(size 1.27 1.27)
-				)
-			)
-		)
-		(property "Description" ""
-			(at 0 0 90)
-			(unlocked yes)
-			(layer "F.Fab")
-			(hide yes)
-			(effects
-				(font
-					(size 1.27 1.27)
-				)
-			)
-		)
-		(sheetname "/")
-		(sheetfile "SparkFun_Artemis_OpenLog.kicad_sch")
-		(units
-			(unit
-				(name "A")
-				(pins "1" "2")
-			)
-		)
-		(attr dnp)
-		(duplicate_pad_numbers_are_jumpers no)
-		(fp_line
-			(start 0.8636 1.016)
-			(end -0.8636 1.016)
-			(stroke
-				(width 0.1524)
-				(type solid)
-			)
-			(layer "F.SilkS")
-		)
-		(fp_line
-			(start -1.1176 0.762)
-			(end -1.1176 -0.762)
-			(stroke
-				(width 0.1524)
-				(type solid)
-			)
-			(layer "F.SilkS")
-		)
-		(fp_line
-			(start 1.1176 0.762)
-			(end 1.1176 -0.762)
-			(stroke
-				(width 0.1524)
-				(type solid)
-			)
-			(layer "F.SilkS")
-		)
-		(fp_line
-			(start -0.8636 -1.016)
-			(end 0.8636 -1.016)
-			(stroke
-				(width 0.1524)
-				(type solid)
-			)
-			(layer "F.SilkS")
-		)
-		(fp_arc
-			(start -0.8636 1.016)
-			(mid -1.043205 0.941605)
-			(end -1.1176 0.762)
-			(stroke
-				(width 0.1524)
-				(type solid)
-			)
-			(layer "F.SilkS")
-		)
-		(fp_arc
-			(start 1.1176 0.762)
-			(mid 1.043205 0.941605)
-			(end 0.8636 1.016)
-			(stroke
-				(width 0.1524)
-				(type solid)
-			)
-			(layer "F.SilkS")
-		)
-		(fp_arc
-			(start -1.1176 -0.762)
-			(mid -1.043205 -0.941605)
-			(end -0.8636 -1.016)
-			(stroke
-				(width 0.1524)
-				(type solid)
-			)
-			(layer "F.SilkS")
-		)
-		(fp_arc
-			(start 0.8636 -1.016)
-			(mid 1.043205 -0.941605)
-			(end 1.1176 -0.762)
-			(stroke
-				(width 0.1524)
-				(type solid)
-			)
-			(layer "F.SilkS")
-		)
-		(pad "1" smd roundrect
-			(at -0.4064 0 270)
-			(size 0.635 1.27)
-			(layers "F.Cu" "F.Mask")
-			(roundrect_rratio 0.08)
-			(net "Net-(U8-(SDA2{slash}SDI2{slash}RX1)~{D25})")
-			(pinfunction "1_1")
-			(pintype "passive")
-			(solder_mask_margin 0.0635)
-			(solder_paste_margin 0)
-			(thermal_bridge_angle 0)
-		)
-		(pad "2" smd roundrect
-			(at 0.4064 0 270)
-			(size 0.635 1.27)
-			(layers "F.Cu" "F.Mask")
-			(roundrect_rratio 0.08)
-			(net "VREG_EN")
-			(pinfunction "2_2")
-			(pintype "passive")
-			(solder_mask_margin 0.0635)
-			(solder_paste_margin 0)
-			(thermal_bridge_angle 0)
-		)
-		(embedded_fonts no)
-	)
 	(footprint "SparkFun-Capacitor:C_0402_1005Metric"
 		(layer "F.Cu")
@@
 			(layers "F.Cu" "F.Mask" "F.Paste")
 			(roundrect_rratio 0.127)
-			(net "Net-(U8-(SDA2{slash}SDI2{slash}RX1)~{D25})")
+			(net "Net-(JP0-A)")
 			(pinfunction "(SDA2/SDI2/RX1)~{D25}_~D25")
 			(pintype "bidirectional")
@@
 		(width 0.1524)
 		(layer "F.Cu")
-		(net "Net-(U8-(SDA2{slash}SDI2{slash}RX1)~{D25})")
+		(net "Net-(JP0-A)")
 	)
 	(segment
@@
 		(width 0.1524)
 		(layer "F.Cu")
-		(net "Net-(U8-(SDA2{slash}SDI2{slash}RX1)~{D25})")
+		(net "Net-(JP0-A)")
 	)
 	(segment
@@
 		(width 0.1524)
 		(layer "F.Cu")
-		(net "Net-(U8-(SDA2{slash}SDI2{slash}RX1)~{D25})")
+		(net "Net-(JP0-A)")
 	)
 	(segment
@@
 		(width 0.1524)
 		(layer "F.Cu")
-		(net "Net-(U8-(SDA2{slash}SDI2{slash}RX1)~{D25})")
+		(net "Net-(JP0-A)")
 	)
 	(segment
@@
 		(width 0.1524)
 		(layer "F.Cu")
-		(net "Net-(U8-(SDA2{slash}SDI2{slash}RX1)~{D25})")
+		(net "Net-(JP0-A)")
 	)
 	(via
@@
 		(drill 0.3048)
 		(layers "F.Cu" "B.Cu")
-		(net "Net-(U8-(SDA2{slash}SDI2{slash}RX1)~{D25})")
+		(net "Net-(JP0-A)")
 	)
 	(via
@@
 		(drill 0.3048)
 		(layers "F.Cu" "B.Cu")
-		(net "Net-(U8-(SDA2{slash}SDI2{slash}RX1)~{D25})")
+		(net "Net-(JP0-A)")
 	)
 	(segment
@@
 		(width 0.1524)
 		(layer "B.Cu")
-		(net "Net-(U8-(SDA2{slash}SDI2{slash}RX1)~{D25})")
+		(net "Net-(JP0-A)")
 	)
 	(segment
@@
 		(width 0.1524)
 		(layer "B.Cu")
-		(net "Net-(U8-(SDA2{slash}SDI2{slash}RX1)~{D25})")
+		(net "Net-(JP0-A)")
 	)
 	(segment

Commit message: Save point (near the end)
Parts:
- removed FRAME1: FRAME-LEDGER, CREATIVE_COMMONS
- removed LOGO3: SPECIAL_INSTRUCTIONS-ORDERING, ORDERING_INSTRUCTIONS
- FID1: renamed from FD1; value FIDUCIAL1X2 -> Fiducial_0.5mm; footprint FIDUCIAL-1X2 -> SparkFun-Aesthetic:Fiducial_0.5mm_Mask1mm
- FID2: renamed from FD2; value FIDUCIAL1X2 -> Fiducial_0.5mm; footprint FIDUCIAL-1X2 -> SparkFun-Aesthetic:Fiducial_0.5mm_Mask1mm
- FID3: renamed from FD3; value FIDUCIAL1X2 -> Fiducial_0.5mm; footprint FIDUCIAL-1X2 -> SparkFun-Aesthetic:Fiducial_0.5mm_Mask1mm
- FID4: renamed from FD4; value FIDUCIAL1X2 -> Fiducial_0.5mm; footprint FIDUCIAL-1X2 -> SparkFun-Aesthetic:Fiducial_0.5mm_Mask1mm
- ST1: renamed from H1; value STAND-OFF -> Standoff; footprint STAND-OFF -> SparkFun-Hardware:Standoff
- ST2: renamed from H2; value STAND-OFF -> Standoff; footprint STAND-OFF -> SparkFun-Hardware:Standoff
- ST3: renamed from H3; value STAND-OFF -> Standoff; footprint STAND-OFF -> SparkFun-Hardware:Standoff
- ST4: renamed from H4; value STAND-OFF -> Standoff; footprint STAND-OFF -> SparkFun-Hardware:Standoff
- U5: footprint LGA-28 -> SparkFun-Semiconductor-Standard:LGA-28_5.2x3.8mm_P0.5mm
- U8: value ARTEMIS_MODULE -> Artemis Module; footprint ARTEMIS_FP -> SparkFun-Semiconductor-Nonstandard:Artemis_Module
- turned U5 to 180 degrees
Connections:
- U10 pad 4: unconnected-(U10-~{RTS}-Pad4) -> ARTEMIS_~{RTS}
- U10 pad 5: ARTEMIS_~{RTS} -> unconnected-(U10-~{CTS}-Pad5)
Other:
- board text added: "Finish: ENIG"
- board text added: "Inner Copper Weight: 0.5oz"
- board text added: "Layers: 4"
- board text added: "Material: TG135"
- board text added: "Ordering Notes"
- board text added: "Outer Copper Weight: 1oz"
- board text added: "Silkscreen Color: White"
- board text added: "Solder Mask: Red"
- board text added: "Thickness: 1.6mm"
- board text removed: "1.6mm thickness"
- board text removed: "4-layer board"
- board text removed: "ENIG finish"
- board text removed: "N. Seidle"

Commit message: Save point
Parts:
- removed LOGO1: SFE_LOGO_NAME.1_INCH, SFE_LOGO_NAME_.1
- removed LOGO2: OSHW-LOGOS, OSHW-LOGO-S
- removed LOGO4, LOGO5: SFE_LOGO_FLAME.1_INCH, SFE_LOGO_FLAME_.1
- added G1: OSHW_Logo, SparkFun-Aesthetic:Creative_Commons_License, F.Cu at (73.2, 160.6)
- added Ref**: Val**, SparkFun-Aesthetic:OSHW_Logo_4mm, B.Cu at (146.9, 116.7)
- TP1: value TEST-POINT3 -> 1.0mm; footprint PAD.03X.03 -> SparkFun-Connector:TestPoint-1.0mm
Connections:
- U5 pad 1: (no net) -> unconnected-(U5-RESV_NC-Pad1)
- U5 pad 12: (no net) -> unconnected-(U5-RESV_NC-Pad12)
- U5 pad 13: (no net) -> unconnected-(U5-RESV_NC-Pad13)
- U5 pad 21: (no net) -> unconnected-(U5-RESV_NC-Pad21)
- U5 pad 22: (no net) -> unconnected-(U5-RESV_NC-Pad22)
- U5 pad 23: (no net) -> unconnected-(U5-RESV_NC-Pad23)
- U5 pad 24: (no net) -> unconnected-(U5-RESV_NC-Pad24)
- U5 pad 7: (no net) -> unconnected-(U5-RESV_NC-Pad7)
- U5 pad 8: (no net) -> unconnected-(U5-RESV_NC-Pad8)

Commit message: Updates microSD - save point
Parts:
- J6: value MICRO-SD -> microSD; footprint MICRO-SD-SOCKET -> SparkFun-Connector:microSD_SOCKET
- moved J6 9.97 mm to (148.5, 100.4)
Connections:
- C46 pad 1: Net-(Q2-D) -> Net-(J6-VDD)
- Q2 pad 3: Net-(Q2-D) -> Net-(J6-VDD)
Routing:
- net Net-(Q2-D): track 13.6 -> 0.00 mm, vias 4 -> 0
- net Net-(J6-VDD): track 0.00 -> 13.6 mm, vias 0 -> 4
